File: PCB/OSHE-Reader-Buck-Converter.kicad_sch (KiCad schematic)
At the start: 17 parts, among them U3 TPS5432DDAR

Commit message: Minor fixes to PCB: schottky diode for battery charging and general battery charging routing fixes
Parts:
- U3: footprint DDA_R-PDSO-G8_TEX -> TPS5432DDAR:DDA_R-PDSO-G8_TEX
